Commit message: Update simulation map and four wheel car

File: zhihui_shequ_ros/src/zhihui_shequ_sim/urdf/smart_car.xacro (robot description, xacro)
@@ -1,52 +1,40 @@
 <?xml version="1.0"?>
 <robot name="smart_car" xmlns:xacro="http://www.ros.org/wiki/xacro">
-  <xacro:property name="base_length" value="0.55"/>
-  <xacro:property name="base_width" value="0.36"/>
+  <xacro:property name="base_length" value="0.68"/>
+  <xacro:property name="base_width" value="0.42"/>
   <xacro:property name="base_height" value="0.16"/>
   <xacro:property name="wheel_radius" value="0.075"/>
   <xacro:property name="wheel_width" value="0.045"/>
-  <xacro:property name="wheel_y" value="0.215"/>
+  <xacro:property name="wheel_y" value="0.245"/>
+  <xacro:property name="front_x" value="0.23"/>
+  <xacro:property name="rear_x" value="-0.23"/>
   <link name="base_footprint"/>
   <joint name="base_joint" type="fixed">
     <parent link="base_footprint"/>
     <child link="base_link"/>
-    <origin xyz="0 0 0.14" rpy="0 0 0"/>
+    <origin xyz="0 0 0.16" rpy="0 0 0"/>
   </joint>
   <link name="base_link">
     <visual>
-      <geometry>
-        <box size="${base_length} ${base_width} ${base_height}"/>
-      </geometry>
-      <material name="blue">
-        <color rgba="0.05 0.22 0.75 1"/>
-      </material>
+      <geometry><box size="${base_length} ${base_width} ${base_height}"/></geometry>
+      <material name="blue"><color rgba="0.05 0.22 0.75 1"/></material>
     </visual>
-    <collision>
-      <geometry>
-        <box size="${base_length} ${base_width} ${base_height}"/>
-      </geometry>
-    </collision>
+    <collision><geometry><box size="${base_length} ${base_width} ${base_height}"/></geometry></collision>
     <inertial>
-      <mass value="6.0"/>
+      <mass value="7.0"/>
       <origin xyz="0 0 0"/>
-      <inertia ixx="0.08" ixy="0" ixz="0" iyy="0.14" iyz="0" izz="0.18"/>
+      <inertia ixx="0.10" ixy="0" ixz="0" iyy="0.18" iyz="0" izz="0.22"/>
     </inertial>
   </link>
-  <xacro:macro name="wheel" params="name y">
+  <xacro:macro name="wheel" params="name x y">
     <link name="${name}">
       <visual>
         <origin rpy="1.5708 0 0"/>
-        <geometry>
-          <cylinder radius="${wheel_radius}" length="${wheel_width}"/>
-        </geometry>
-        <material name="dark">
-          <color rgba="0.02 0.02 0.02 1"/>
-        </material>
+        <geometry><cylinder radius="${wheel_radius}" length="${wheel_width}"/></geometry>
+        <material name="dark"><color rgba="0.02 0.02 0.02 1"/></material>
       </visual>
       <collision>
         <origin rpy="1.5708 0 0"/>
-        <geometry>
-          <cylinder radius="${wheel_radius}" length="${wheel_width}"/>
-        </geometry>
+        <geometry><cylinder radius="${wheel_radius}" length="${wheel_width}"/></geometry>
       </collision>
       <inertial>
@@ -59,49 +47,18 @@
       <parent link="base_link"/>
       <child link="${name}"/>
-      <origin xyz="0 ${y} -0.065" rpy="0 0 0"/>
+      <origin xyz="${x} ${y} -0.075" rpy="0 0 0"/>
       <axis xyz="0 1 0"/>
     </joint>
   </xacro:macro>
-  <xacro:wheel name="left_wheel" y="${wheel_y}"/>
-  <xacro:wheel name="right_wheel" y="-${wheel_y}"/>
-  <link name="caster_link">
-    <visual>
-      <geometry>
-        <sphere radius="0.045"/>
-      </geometry>
-      <material name="gray">
-        <color rgba="0.45 0.45 0.45 1"/>
-      </material>
-    </visual>
-    <collision>
-      <geometry>
-        <sphere radius="0.045"/>
-      </geometry>
-    </collision>
-    <inertial>
-      <mass value="0.1"/>
-      <origin xyz="0 0 0"/>
-      <inertia ixx="0.0001" ixy="0" ixz="0" iyy="0.0001" iyz="0" izz="0.0001"/>
-    </inertial>
-  </link>
-  <joint name="caster_joint" type="fixed">
-    <parent link="base_link"/>
-    <child link="caster_link"/>
-    <origin xyz="-0.22 0 -0.085" rpy="0 0 0"/>
-  </joint>
+  <xacro:wheel name="left_front_wheel" x="${front_x}" y="${wheel_y}"/>
+  <xacro:wheel name="left_rear_wheel" x="${rear_x}" y="${wheel_y}"/>
+  <xacro:wheel name="right_front_wheel" x="${front_x}" y="-${wheel_y}"/>
+  <xacro:wheel name="right_rear_wheel" x="${rear_x}" y="-${wheel_y}"/>
   <link name="camera_link">
     <visual>
-      <geometry>
-        <box size="0.08 0.09 0.06"/>
-      </geometry>
-      <material name="black">
-        <color rgba="0.01 0.01 0.01 1"/>
-      </material>
+      <geometry><box size="0.08 0.09 0.06"/></geometry>
+      <material name="black"><color rgba="0.01 0.01 0.01 1"/></material>
     </visual>
-    <collision>
-      <geometry>
-        <box size="0.08 0.09 0.06"/>
-      </geometry>
-    </collision>
+    <collision><geometry><box size="0.08 0.09 0.06"/></geometry></collision>
     <inertial>
       <mass value="0.1"/>
@@ -113,15 +70,11 @@
     <parent link="base_link"/>
     <child link="camera_link"/>
-    <origin xyz="0.28 0 0.12" rpy="0 0 0"/>
+    <origin xyz="0.36 0 0.13" rpy="0 0 0"/>
   </joint>
-  <gazebo reference="base_link">
-    <material>Gazebo/Blue</material>
-  </gazebo>
-  <gazebo reference="left_wheel">
-    <material>Gazebo/Black</material>
-  </gazebo>
-  <gazebo reference="right_wheel">
-    <material>Gazebo/Black</material>
-  </gazebo>
+  <gazebo reference="base_link"><material>Gazebo/Blue</material></gazebo>
+  <gazebo reference="left_front_wheel"><material>Gazebo/Black</material></gazebo>
+  <gazebo reference="left_rear_wheel"><material>Gazebo/Black</material></gazebo>
+  <gazebo reference="right_front_wheel"><material>Gazebo/Black</material></gazebo>
+  <gazebo reference="right_rear_wheel"><material>Gazebo/Black</material></gazebo>
   <gazebo>
     <plugin name="differential_drive_controller" filename="libgazebo_ros_diff_drive.so">
@@ -133,10 +86,10 @@
       <publishOdomTF>true</publishOdomTF>
       <publishWheelJointState>true</publishWheelJointState>
-      <leftJoint>left_wheel_joint</leftJoint>
-      <rightJoint>right_wheel_joint</rightJoint>
-      <wheelSeparation>0.43</wheelSeparation>
+      <leftJoint>left_rear_wheel_joint</leftJoint>
+      <rightJoint>right_rear_wheel_joint</rightJoint>
+      <wheelSeparation>0.49</wheelSeparation>
       <wheelDiameter>0.15</wheelDiameter>
       <wheelAcceleration>2.0</wheelAcceleration>
-      <wheelTorque>8.0</wheelTorque>
+      <wheelTorque>10.0</wheelTorque>
       <updateRate>50</updateRate>
     </plugin>
@@ -150,13 +103,6 @@
       <camera name="front_camera">
         <horizontal_fov>1.047</horizontal_fov>
-        <image>
-          <width>640</width>
-          <height>480</height>
-          <format>R8G8B8</format>
-        </image>
-        <clip>
-          <near>0.05</near>
-          <far>30</far>
-        </clip>
+        <image><width>640</width><height>480</height><format>R8G8B8</format></image>
+        <clip><near>0.05</near><far>30</far></clip>
       </camera>
       <plugin name="front_camera_controller" filename="libgazebo_ros_camera.so">

Commit message: Reset Gazebo car spawn and improve visibility

File: zhihui_shequ_ros/src/zhihui_shequ_sim/urdf/smart_car.xacro (robot description, xacro)
@@ -19,4 +19,14 @@
       <geometry><box size="${base_length} ${base_width} ${base_height}"/></geometry>
       <material name="blue"><color rgba="0.05 0.22 0.75 1"/></material>
+    </visual>
+    <visual name="visibility_mast">
+      <origin xyz="-0.18 0 0.36" rpy="0 0 0"/>
+      <geometry><cylinder radius="0.025" length="0.72"/></geometry>
+      <material name="bright_orange"><color rgba="1.0 0.35 0.0 1"/></material>
+    </visual>
+    <visual name="visibility_flag">
+      <origin xyz="-0.18 0.12 0.72" rpy="0 0 0"/>
+      <geometry><box size="0.28 0.035 0.18"/></geometry>
+      <material name="bright_yellow"><color rgba="1.0 0.9 0.05 1"/></material>
     </visual>
     <collision><geometry><box size="${base_length} ${base_width} ${base_height}"/></geometry></collision>

Commit message: Drive mission route with Gazebo model state

File: zhihui_shequ_ros/src/zhihui_shequ_sim/urdf/smart_car.xacro (robot description, xacro)
@@ -37,5 +37,5 @@
     </inertial>
   </link>
-  <xacro:macro name="wheel" params="name x y">
+  <xacro:macro name="drive_wheel" params="name x y">
     <link name="${name}">
       <visual>
@@ -61,8 +61,27 @@
     </joint>
   </xacro:macro>
-  <xacro:wheel name="left_front_wheel" x="${front_x}" y="${wheel_y}"/>
-  <xacro:wheel name="left_rear_wheel" x="${rear_x}" y="${wheel_y}"/>
-  <xacro:wheel name="right_front_wheel" x="${front_x}" y="-${wheel_y}"/>
-  <xacro:wheel name="right_rear_wheel" x="${rear_x}" y="-${wheel_y}"/>
+  <xacro:macro name="visual_wheel" params="name x y">
+    <link name="${name}">
+      <visual>
+        <origin rpy="1.5708 0 0"/>
+        <geometry><cylinder radius="${wheel_radius}" length="${wheel_width}"/></geometry>
+        <material name="dark"><color rgba="0.02 0.02 0.02 1"/></material>
+      </visual>
+      <inertial>
+        <mass value="0.05"/>
+        <origin xyz="0 0 0"/>
+        <inertia ixx="0.0001" ixy="0" ixz="0" iyy="0.0001" iyz="0" izz="0.0001"/>
+      </inertial>
+    </link>
+    <joint name="${name}_joint" type="fixed">
+      <parent link="base_link"/>
+      <child link="${name}"/>
+      <origin xyz="${x} ${y} -0.075" rpy="0 0 0"/>
+    </joint>
+  </xacro:macro>
+  <xacro:visual_wheel name="left_front_wheel" x="${front_x}" y="${wheel_y}"/>
+  <xacro:drive_wheel name="left_rear_wheel" x="${rear_x}" y="${wheel_y}"/>
+  <xacro:visual_wheel name="right_front_wheel" x="${front_x}" y="-${wheel_y}"/>
+  <xacro:drive_wheel name="right_rear_wheel" x="${rear_x}" y="-${wheel_y}"/>
   <link name="camera_link">
     <visual>

Commit message: Save current simulation state

File: zhihui_shequ_ros/src/zhihui_shequ_sim/urdf/smart_car.xacro (robot description, xacro)
@@ -6,4 +6,5 @@
   <xacro:property name="wheel_radius" value="0.075"/>
   <xacro:property name="wheel_width" value="0.045"/>
+  <xacro:property name="wheel_z" value="-0.035"/>
   <xacro:property name="wheel_y" value="0.245"/>
   <xacro:property name="front_x" value="0.23"/>
@@ -57,5 +58,5 @@
       <parent link="base_link"/>
       <child link="${name}"/>
-      <origin xyz="${x} ${y} -0.075" rpy="0 0 0"/>
+      <origin xyz="${x} ${y} ${wheel_z}" rpy="0 0 0"/>
       <axis xyz="0 1 0"/>
     </joint>
@@ -68,4 +69,8 @@
         <material name="dark"><color rgba="0.02 0.02 0.02 1"/></material>
       </visual>
+      <collision>
+        <origin rpy="1.5708 0 0"/>
+        <geometry><cylinder radius="${wheel_radius}" length="${wheel_width}"/></geometry>
+      </collision>
       <inertial>
         <mass value="0.05"/>
@@ -77,10 +82,10 @@
       <parent link="base_link"/>
       <child link="${name}"/>
-      <origin xyz="${x} ${y} -0.075" rpy="0 0 0"/>
+      <origin xyz="${x} ${y} ${wheel_z}" rpy="0 0 0"/>
     </joint>
   </xacro:macro>
-  <xacro:visual_wheel name="left_front_wheel" x="${front_x}" y="${wheel_y}"/>
+  <xacro:drive_wheel name="left_front_wheel" x="${front_x}" y="${wheel_y}"/>
   <xacro:drive_wheel name="left_rear_wheel" x="${rear_x}" y="${wheel_y}"/>
-  <xacro:visual_wheel name="right_front_wheel" x="${front_x}" y="-${wheel_y}"/>
+  <xacro:drive_wheel name="right_front_wheel" x="${front_x}" y="-${wheel_y}"/>
   <xacro:drive_wheel name="right_rear_wheel" x="${rear_x}" y="-${wheel_y}"/>
   <link name="camera_link">
