Commit message: Add SLAM and autonomous navigation stack

File: zhihui_shequ_ros/src/zhihui_shequ_sim/urdf/smart_car.xacro (robot description, xacro)
@@ -106,4 +106,21 @@
     <origin xyz="0.36 0 0.13" rpy="0 0 0"/>
   </joint>
+  <link name="lidar_link">
+    <visual>
+      <geometry><cylinder radius="0.055" length="0.06"/></geometry>
+      <material name="lidar_gray"><color rgba="0.22 0.24 0.27 1"/></material>
+    </visual>
+    <collision><geometry><cylinder radius="0.055" length="0.06"/></geometry></collision>
+    <inertial>
+      <mass value="0.12"/>
+      <origin xyz="0 0 0"/>
+      <inertia ixx="0.00008" ixy="0" ixz="0" iyy="0.00008" iyz="0" izz="0.00012"/>
+    </inertial>
+  </link>
+  <joint name="lidar_joint" type="fixed">
+    <parent link="base_link"/>
+    <child link="lidar_link"/>
+    <origin xyz="0.02 0 0.18" rpy="0 0 0"/>
+  </joint>
   <gazebo reference="base_link"><material>Gazebo/Blue</material></gazebo>
   <gazebo reference="left_front_wheel"><material>Gazebo/Black</material></gazebo>
@@ -111,4 +128,5 @@
   <gazebo reference="right_front_wheel"><material>Gazebo/Black</material></gazebo>
   <gazebo reference="right_rear_wheel"><material>Gazebo/Black</material></gazebo>
+  <gazebo reference="lidar_link"><material>Gazebo/DarkGrey</material></gazebo>
   <gazebo>
     <plugin name="differential_drive_controller" filename="libgazebo_ros_diff_drive.so">
@@ -117,4 +135,5 @@
       <odometryTopic>odom</odometryTopic>
       <odometryFrame>odom</odometryFrame>
+      <odometrySource>world</odometrySource>
       <robotBaseFrame>base_footprint</robotBaseFrame>
       <publishWheelTF>false</publishWheelTF>
@@ -151,3 +170,35 @@
     </sensor>
   </gazebo>
+  <gazebo reference="lidar_link">
+    <sensor type="ray" name="smart_car_360_lidar">
+      <always_on>true</always_on>
+      <visualize>true</visualize>
+      <update_rate>10.0</update_rate>
+      <ray>
+        <scan>
+          <horizontal>
+            <samples>720</samples>
+            <resolution>1</resolution>
+            <min_angle>-3.14159265</min_angle>
+            <max_angle>3.14159265</max_angle>
+          </horizontal>
+        </scan>
+        <range>
+          <min>0.12</min>
+          <max>12.0</max>
+          <resolution>0.01</resolution>
+        </range>
+        <noise>
+          <type>gaussian</type>
+          <mean>0.0</mean>
+          <stddev>0.005</stddev>
+        </noise>
+      </ray>
+      <plugin name="smart_car_lidar_controller" filename="libgazebo_ros_laser.so">
+        <robotNamespace>/</robotNamespace>
+        <topicName>/scan</topicName>
+        <frameName>lidar_link</frameName>
+      </plugin>
+    </sensor>
+  </gazebo>
 </robot>
